Commit message: Sửa hình học URDF: thân lộn ngược, box sai trục, hình vẽ trùng lặp
Ba lỗi trong generate_urdf.py làm model hiện sai dù nạp được:

- Thân và đầu treo xuống dưới khớp như tay chân, nên thân nằm dưới eo
  và hình chỉ cao 1,53 m. Giờ hai đoạn này dựng lên trên khớp.
- Box xuất theo thứ tự (rộng, sâu, cao) vào (x, y, z), trong khi URDF lấy
  x là hướng trước: bàn chân, pelvis, thân, đầu bị xoay 90°, và tensor
  quán tính tính theo trục sai. Giờ theo đúng quy ước x trước, y trái.
- 16 link trung gian chép nguyên hình và collision của đoạn kế tiếp.
  Giờ chúng chỉ mang 1 g, không có hình; mỗi đoạn vẽ đúng một lần.

Audit cũ chỉ cộng chiều dài khai báo nên báo "1.75 ok" trên model lộn
ngược. Thêm bốn kiểm tra đo trên hình thật (chiều cao vẽ, số đoạn vẽ,
thân trên eo, bàn chân hướng trước); cả bốn bắt được lỗi trên file cũ.

Co-Authored-By: Claude Opus 5.5 <noreply@anthropic.com>

File: hardware/sim-model/gems.urdf (robot description, URDF)
Before this commit: robot gems, 31 links, 30 joints
Links:
- link head: geometry collision box size=0.1900 0.1600 0.2200; visual box size=0.1900 0.1600 0.2200
- link l_ankle_pitch_link: geometry 
- link l_foot: geometry collision box size=0.2600 0.1000 0.0700; visual box size=0.2600 0.1000 0.0700
- link l_hip_pitch_link: geometry 
- link l_hip_roll_link: geometry 
- link l_shoulder_pitch_link: geometry 
- link l_shoulder_roll_link: geometry 
- link l_wrist_pitch_link: geometry 
- link l_wrist_yaw_link: geometry 
- link neck_yaw_link: geometry 
- link pelvis: geometry collision box size=0.1800 0.3000 0.1600; visual box size=0.1800 0.3000 0.1600
- link r_ankle_pitch_link: geometry 
- link r_foot: geometry collision box size=0.2600 0.1000 0.0700; visual box size=0.2600 0.1000 0.0700
- link r_hip_pitch_link: geometry 
- link r_hip_roll_link: geometry 
- link r_shoulder_pitch_link: geometry 
- link r_shoulder_roll_link: geometry 
- link r_wrist_pitch_link: geometry 
- link r_wrist_yaw_link: geometry 
- link torso: geometry collision box size=0.2100 0.3400 0.4600; visual box size=0.2100 0.3400 0.4600
- link waist_yaw_link: geometry 

Commit message: Sửa chiều khớp URDF: khuỷu gập ra sau, cổ chân đảo, bên phải không đối xứng
Đo bằng forward kinematics (quy ước URDF: x trước, y trái):

- Khuỷu tay gập ra sau: giới hạn (0, 2.62) quanh +y đưa cẳng tay về -x.
  Đổi thành (-2.62, 0). Đây là lý do mặt trước trông như mặt sau, và
  khớp vai (vốn đúng) trông như bị ngược.
- Cổ chân đảo biên độ: gập mu 50°, gập gan 30°. Đổi thành gập gan 50°,
  gập mu 30°.
- Giới hạn roll và yaw dùng chung cho hai bên, không lấy đối xứng: tay
  phải dạng xuyên qua thân, hai hông dạng không đều. Bên phải giờ được
  lấy đối xứng qua mặt phẳng dọc. Dạng hông 45°, khép 30°.

Audit thêm "joints move as named": đưa từng khớp tới giới hạn ở cả hai
bên, kiểm tra hướng và biên độ bằng FK. Thử lật ngược từng khớp chi
(vai, khuỷu, hông, gối, cổ chân, roll) và bỏ phần đối xứng: đều bị bắt.

Co-Authored-By: Claude Opus 5.5 <noreply@anthropic.com>

File: hardware/sim-model/gems.urdf (robot description, URDF)
Before this commit: robot gems, 31 links, 30 joints
Joints:
- joint l_ankle_pitch: limit lower=-0.8700 upper=0.5200 effort=200.0 velocity=8.0 -> lower=-0.5200 upper=0.8700 effort=200.0 velocity=8.0
- joint l_elbow: limit lower=0.0000 upper=2.6200 effort=200.0 velocity=8.0 -> lower=-2.6200 upper=0.0000 effort=200.0 velocity=8.0
- joint l_hip_roll: limit lower=-0.7900 upper=0.5200 effort=200.0 velocity=8.0 -> lower=-0.5200 upper=0.7900 effort=200.0 velocity=8.0
- joint r_ankle_pitch: limit lower=-0.8700 upper=0.5200 effort=200.0 velocity=8.0 -> lower=-0.5200 upper=0.8700 effort=200.0 velocity=8.0
- joint r_elbow: limit lower=0.0000 upper=2.6200 effort=200.0 velocity=8.0 -> lower=-2.6200 upper=0.0000 effort=200.0 velocity=8.0
- joint r_shoulder_roll: limit lower=-0.3500 upper=3.1400 effort=200.0 velocity=8.0 -> lower=-3.1400 upper=0.3500 effort=200.0 velocity=8.0

Commit message: D-9: cột sống liên động ba đoạn, trục nghiêng bên, biên khớp theo cơ cấu
Anh Plone duyệt ba việc.

- D-9: thân là cột sống ba đoạn (thắt lưng, ngực dưới, ngực trên mang vai,
  cổ và pack). Mỗi trục xoay, gập, nghiêng bên có một actuator; cơ cấu liên
  động chia chuyển động cho cả ba đoạn. Lý do: người xoay chủ yếu ở đoạn
  ngực, thắt lưng gần như không xoay, còn một khớp eo đơn thì xoay đúng chỗ
  người không xoay. Phương án một actuator cho mỗi đoạn (kiểu Kotaro,
  Kenshiro) bị loại vì khó điều khiển, chịu tải kém và vượt ngân sách f_act.
- Thêm trục nghiêng bên: khớp chính từ 30 thành 31, khớp ghi log từ 40
  thành 41. Log full tier là 328 kB/s, 2,6 Mbps, 1,18 GB/h. Đã cập nhật spec
  05, 06, 07, gems_budget và conformance-record. Mô-men của trục nghiêng bên
  chưa suy ra được: f_act vẫn tính trên 30 khớp đã sizing, và điều này được
  ghi rõ ở kinematics, spec 02.6, sizing và BOM.
- Biên độ khớp theo cơ cấu, không theo sinh học (kinematics §1.5): vai
  250°/220°, khuỷu 200°, gập hông 210°, gối 200° (khoá ở 0° riêng, phải là
  phanh lò xo tự đóng khi mất điện), xoay thân 180° chia ba đoạn, nghiêng
  bên 90° (tạm), cổ giữ nguyên.
- URDF: 3 đoạn thân, khớp theo dùng <mimic>; <limit> là biên cơ khí,
  <safety_controller> là biên mềm giống người. Audit thêm ba kiểm tra (31
  khớp, thân chia đủ ba đoạn, biên cơ khí bao trọn biên mềm). Các kiểm tra
  bất đối xứng kiểu người chạy trên biên mềm. yourdfpy và urdf-loader đều
  nạp được; FK xác nhận thân xoay 30/60/90°.
- BOM: đổi tên waist thành trunk, thêm module trunk_roll, hai đoạn khung
  cột sống và cơ cấu liên động (MBOM 494 thao tác, 59 routing).

Co-Authored-By: Claude Opus 5.5 <noreply@anthropic.com>

File: hardware/sim-model/gems.urdf (robot description, URDF)
Before this commit: robot gems, 31 links, 30 joints
Links:
- removed link waist_yaw_link
- added link spine_lumbar, mass 12.0391; collision box size=0.2100 0.3400 0.1200; visual box size=0.2100 0.3400 0.1200
- added link spine_thoracic, mass 12.0391; collision box size=0.2100 0.3400 0.1200; visual box size=0.2100 0.3400 0.1200
- added link trunk_pitch_2_link, mass 0.0010
- added link trunk_pitch_3_link, mass 0.0010
- added link trunk_pitch_link, mass 0.0010
- added link trunk_yaw_2_link, mass 0.0010
- added link trunk_yaw_3_link, mass 0.0010
- added link trunk_yaw_link, mass 0.0010
- link torso: mass 46.1500 -> 22.0717; geometry collision box size=0.2100 0.3400 0.2200; visual box size=0.2100 0.3400 0.2200
Joints:
- removed joint waist_pitch
- removed joint waist_yaw
- added joint trunk_pitch: type revolute, parent trunk_yaw_link, child trunk_pitch_link, origin xyz=0 0 0 rpy=0 0 0, axis 0 1 0, limit lower=-0.1733 upper=0.3500 effort=200.0 velocity=8.0
- added joint trunk_pitch_2: type revolute, parent trunk_yaw_2_link, child trunk_pitch_2_link, origin xyz=0 0 0 rpy=0 0 0, axis 0 1 0, limit lower=-0.1733 upper=0.3500 effort=200.0 velocity=8.0, mimic joint=trunk_pitch multiplier=1 offset=0
- added joint trunk_pitch_3: type revolute, parent trunk_yaw_3_link, child trunk_pitch_3_link, origin xyz=0 0 0 rpy=0 0 0, axis 0 1 0, limit lower=-0.1733 upper=0.3500 effort=200.0 velocity=8.0, mimic joint=trunk_pitch multiplier=1 offset=0
- added joint trunk_roll: type revolute, parent trunk_pitch_link, child spine_lumbar, origin xyz=0 0 0 rpy=0 0 0, axis 1 0 0, limit lower=-0.2633 upper=0.2633 effort=200.0 velocity=8.0
- added joint trunk_roll_2: type revolute, parent trunk_pitch_2_link, child spine_thoracic, origin xyz=0 0 0 rpy=0 0 0, axis 1 0 0, limit lower=-0.2633 upper=0.2633 effort=200.0 velocity=8.0, mimic joint=trunk_roll multiplier=1 offset=0
- added joint trunk_roll_3: type revolute, parent trunk_pitch_3_link, child torso, origin xyz=0 0 0 rpy=0 0 0, axis 1 0 0, limit lower=-0.2633 upper=0.2633 effort=200.0 velocity=8.0, mimic joint=trunk_roll multiplier=1 offset=0
- added joint trunk_yaw: type revolute, parent pelvis, child trunk_yaw_link, origin xyz=0 0 0.0000 rpy=0 0 0, axis 0 0 1, limit lower=-0.5233 upper=0.5233 effort=200.0 velocity=8.0
- added joint trunk_yaw_2: type revolute, parent spine_lumbar, child trunk_yaw_2_link, origin xyz=0 0 0.1200 rpy=0 0 0, axis 0 0 1, limit lower=-0.5233 upper=0.5233 effort=200.0 velocity=8.0, mimic joint=trunk_yaw multiplier=1 offset=0
- added joint trunk_yaw_3: type revolute, parent spine_thoracic, child trunk_yaw_3_link, origin xyz=0 0 0.1200 rpy=0 0 0, axis 0 0 1, limit lower=-0.5233 upper=0.5233 effort=200.0 velocity=8.0, mimic joint=trunk_yaw multiplier=1 offset=0
- joint l_elbow: limit lower=-2.6200 upper=0.0000 effort=200.0 velocity=8.0 -> lower=-2.6200 upper=0.8700 effort=200.0 velocity=8.0
- joint l_hip_pitch: limit lower=-2.0900 upper=0.5200 effort=200.0 velocity=8.0 -> lower=-2.0900 upper=1.5700 effort=200.0 velocity=8.0
- joint l_knee: limit lower=0.0000 upper=2.4400 effort=200.0 velocity=8.0 -> lower=-1.0500 upper=2.4400 effort=200.0 velocity=8.0
- joint l_shoulder_pitch: limit lower=-3.1400 upper=1.0500 effort=200.0 velocity=8.0 -> lower=-3.1400 upper=1.2200 effort=200.0 velocity=8.0; origin xyz=0 0.2000 0.4600 rpy=0 0 0 -> xyz=0 0.2000 0.2200 rpy=0 0 0
- joint l_shoulder_roll: limit lower=-0.3500 upper=3.1400 effort=200.0 velocity=8.0 -> lower=-0.7000 upper=3.1400 effort=200.0 velocity=8.0
- joint neck_yaw: origin xyz=0 0 0.4600 rpy=0 0 0 -> xyz=0 0 0.2200 rpy=0 0 0
- joint r_elbow: limit lower=-2.6200 upper=0.0000 effort=200.0 velocity=8.0 -> lower=-2.6200 upper=0.8700 effort=200.0 velocity=8.0
- joint r_hip_pitch: limit lower=-2.0900 upper=0.5200 effort=200.0 velocity=8.0 -> lower=-2.0900 upper=1.5700 effort=200.0 velocity=8.0
- joint r_knee: limit lower=0.0000 upper=2.4400 effort=200.0 velocity=8.0 -> lower=-1.0500 upper=2.4400 effort=200.0 velocity=8.0
- joint r_shoulder_pitch: limit lower=-3.1400 upper=1.0500 effort=200.0 velocity=8.0 -> lower=-3.1400 upper=1.2200 effort=200.0 velocity=8.0; origin xyz=0 -0.2000 0.4600 rpy=0 0 0 -> xyz=0 -0.2000 0.2200 rpy=0 0 0
- joint r_shoulder_roll: limit lower=-3.1400 upper=0.3500 effort=200.0 velocity=8.0 -> lower=-3.1400 upper=0.7000 effort=200.0 velocity=8.0

Commit message: D-8: điểm tham chiếu 2 giờ kèm dock, cao 1,65 m; gói dock DK; giáp giữ 65% chờ bàn
Thân 129,3 → 96,2 kg, γ 3,38 → 2,60, pin 10,3 → 3,9 kWh, hông 229 → 170 Nm,
chân còn 29 kg sức mang so với AKH70-48. Chiều cao 1,65 m: diện tích da 1,6 m²,
đoạn chi và URDF co theo (tầm với 0,66 m, đòn bẩy tâm nắm 0,61 m), giáp 65%
còn 6,2–9,4 kg, taxel ~460.000 và tổng thô 15,1 Gbps ở spec 05. gems_budget
mặc định 2 h, kiểm 93 con số kể cả REF_MASS của script cỡ khớp; spec 00, 02,
03, 05, README, kinematics, plan, BOM, mô hình mô phỏng, hồ sơ conformance
cập nhật. Thêm gói DK-1…DK-5 cho dock vì 2 h chỉ có nghĩa khi có dock.

Co-Authored-By: Claude Fable 5.1 <noreply@anthropic.com>

File: hardware/sim-model/gems.urdf (robot description, URDF)
Before this commit: robot gems, 38 links, 37 joints
Links:
- link head: mass 10.5300 -> 7.7922; geometry collision box size=0.1800 0.1500 0.2100; visual box size=0.1800 0.1500 0.2100
- link l_foot: mass 1.8850 -> 1.3949; geometry collision box size=0.2500 0.0950 0.0660; visual box size=0.2500 0.0950 0.0660
- link l_forearm: mass 2.0800 -> 1.5392; geometry collision cylinder length=0.2500 radius=0.0380; visual cylinder length=0.2500 radius=0.0380
- link l_hand: mass 0.7800 -> 0.5772; geometry collision box size=0.0850 0.0400 0.1100; visual box size=0.0850 0.0400 0.1100
- link l_shank: mass 6.0450 -> 4.4733; geometry collision cylinder length=0.4000 radius=0.0470; visual cylinder length=0.4000 radius=0.0470
- link l_thigh: mass 13.0000 -> 9.6200; geometry collision cylinder length=0.4000 radius=0.0580; visual cylinder length=0.4000 radius=0.0580
- link l_upper_arm: mass 3.6400 -> 2.6936; geometry collision cylinder length=0.3000 radius=0.0450; visual cylinder length=0.3000 radius=0.0450
- link pelvis: mass 18.4600 -> 13.6604; geometry collision box size=0.1700 0.2800 0.1500; visual box size=0.1700 0.2800 0.1500
- link r_foot: mass 1.8850 -> 1.3949; geometry collision box size=0.2500 0.0950 0.0660; visual box size=0.2500 0.0950 0.0660
- link r_forearm: mass 2.0800 -> 1.5392; geometry collision cylinder length=0.2500 radius=0.0380; visual cylinder length=0.2500 radius=0.0380
- link r_hand: mass 0.7800 -> 0.5772; geometry collision box size=0.0850 0.0400 0.1100; visual box size=0.0850 0.0400 0.1100
- link r_shank: mass 6.0450 -> 4.4733; geometry collision cylinder length=0.4000 radius=0.0470; visual cylinder length=0.4000 radius=0.0470
- link r_thigh: mass 13.0000 -> 9.6200; geometry collision cylinder length=0.4000 radius=0.0580; visual cylinder length=0.4000 radius=0.0580
- link r_upper_arm: mass 3.6400 -> 2.6936; geometry collision cylinder length=0.3000 radius=0.0450; visual cylinder length=0.3000 radius=0.0450
- link spine_lumbar: mass 12.0391 -> 8.7363; geometry collision box size=0.2000 0.3200 0.1100; visual box size=0.2000 0.3200 0.1100
- link spine_thoracic: mass 12.0391 -> 8.7363; geometry collision box size=0.2000 0.3200 0.1100; visual box size=0.2000 0.3200 0.1100
- link torso: mass 22.0717 -> 16.6784; geometry collision box size=0.2000 0.3200 0.2100; visual box size=0.2000 0.3200 0.2100
Joints:
- joint l_ankle_pitch: origin xyz=0 0 -0.4200 rpy=0 0 0 -> xyz=0 0 -0.4000 rpy=0 0 0
- joint l_elbow: origin xyz=0 0 -0.3200 rpy=0 0 0 -> xyz=0 0 -0.3000 rpy=0 0 0
- joint l_hip_roll: origin xyz=0 0.0900 -0.1600 rpy=0 0 0 -> xyz=0 0.0900 -0.1500 rpy=0 0 0
- joint l_knee: origin xyz=0 0 -0.4200 rpy=0 0 0 -> xyz=0 0 -0.4000 rpy=0 0 0
- joint l_shoulder_pitch: origin xyz=0 0.2000 0.2200 rpy=0 0 0 -> xyz=0 0.1900 0.2100 rpy=0 0 0
- joint l_wrist_yaw: origin xyz=0 0 -0.2600 rpy=0 0 0 -> xyz=0 0 -0.2500 rpy=0 0 0
- joint neck_yaw: origin xyz=0 0 0.2200 rpy=0 0 0 -> xyz=0 0 0.2100 rpy=0 0 0
- joint r_ankle_pitch: origin xyz=0 0 -0.4200 rpy=0 0 0 -> xyz=0 0 -0.4000 rpy=0 0 0
- joint r_elbow: origin xyz=0 0 -0.3200 rpy=0 0 0 -> xyz=0 0 -0.3000 rpy=0 0 0
- joint r_hip_roll: origin xyz=0 -0.0900 -0.1600 rpy=0 0 0 -> xyz=0 -0.0900 -0.1500 rpy=0 0 0
- joint r_knee: origin xyz=0 0 -0.4200 rpy=0 0 0 -> xyz=0 0 -0.4000 rpy=0 0 0
- joint r_shoulder_pitch: origin xyz=0 -0.2000 0.2200 rpy=0 0 0 -> xyz=0 -0.1900 0.2100 rpy=0 0 0
- joint r_wrist_yaw: origin xyz=0 0 -0.2600 rpy=0 0 0 -> xyz=0 0 -0.2500 rpy=0 0 0
- joint trunk_yaw_2: origin xyz=0 0 0.1200 rpy=0 0 0 -> xyz=0 0 0.1100 rpy=0 0 0
- joint trunk_yaw_3: origin xyz=0 0 0.1200 rpy=0 0 0 -> xyz=0 0 0.1100 rpy=0 0 0
